File: Wirkschaltschema_BMW_R80_7/Wirkschaltschema_BMW_R80_7.kicad_sch (KiCad schematic)
At the start: 10 parts, among them SW1 TURN_R, SW2 TURN_L, SW3 START, SW4 HORN, SW5 BRAKE

Commit message: Symbole erstellt
Parts:
- added LiMa-Kontroller1: ~, symbol Silent_Hektik_LiMa_Dauer_Drehstr._Kont_3Pha.:LiMa
- added Microlino_Zündung1: ~, symbol Silen_Hektik_Microlino Zündung:Silent_Hektik_Microlino_Zündung
Changed lines of the file:
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@@
+	)
+	(symbol
+		(lib_id "Silen_Hektik_Microlino Zündung:Silent_Hektik_Microlino_Zündung")
+		(at 167.64 128.27 0)
+		(unit 1)
+		(exclude_from_sim no)
+		(in_bom yes)
+		(on_board yes)
+		(dnp no)
+		(fields_autoplaced yes)
+		(property "Reference" "Microlino_Zündung1"
+			(at 173.99 142.8749 0)
+			(effects
+				(font
+					(size 1.27 1.27)
+				)
+				(justify left)
+			)
+		)
+		(property "Value" "~"
+			(at 173.99 144.78 0)
+			(effects
+				(font
+					(size 1.27 1.27)
+				)
+				(justify left)
+			)
+		)
+		(property "Footprint" ""
+			(at 167.64 128.27 0)
+			(effects
+				(font
+					(size 1.27 1.27)
+				)
+				(hide yes)
+			)
+		)
+		(property "Datasheet" ""
+			(at 167.64 128.27 0)
+			(effects
+				(font
+					(size 1.27 1.27)
+				)
+				(hide yes)
+			)
+		)
+		(property "Description" ""
+			(at 167.64 128.27 0)
+			(effects
+				(font
+					(size 1.27 1.27)
+				)
+				(hide yes)
+			)
+		)
+		(pin ""
+		)
+		(pin "2"
+		)
+		(pin ""
+		)
+		(pin ""
+		)
+		(pin ""
+		)
+		(pin ""
+		)
+		(pin ""
+		)
+		(pin "1"
+		)
+		(instances
+			(project ""
+				(path "/6b7edb0b-ba84-49d7-8a33-d453b93ff911"
+					(reference "Microlino_Zündung1")
+					(unit 1)
+				)
+			)
+		)
 	)
 	(symbol
@@
 					(unit 1)
 				)
+			)
+		)
+	)
+	(symbol
+		(lib_id "Silent_Hektik_LiMa_Dauer_Drehstr._Kont_3Pha.:LiMa")
+		(at 102.87 135.89 0)
+		(unit 1)
+		(exclude_from_sim no)
+		(in_bom yes)
+		(on_board yes)
+		(dnp no)
+		(fields_autoplaced yes)
+		(property "Reference" "LiMa-Kontroller1"
+			(at 121.92 147.9549 0)
+			(effects
+				(font
+					(size 1.27 1.27)
+				)
+				(justify left)
+			)
+		)
+		(property "Value" "~"
+			(at 121.92 149.86 0)
+			(effects
+				(font
+					(size 1.27 1.27)
+				)
+				(justify left)
+			)
+		)
+		(property "Footprint" ""
+			(at 102.87 135.89 0)
+			(effects
+				(font
+					(size 1.27 1.27)
+				)
+				(hide yes)
+			)
+		)
+		(property "Datasheet" ""
+			(at 102.87 135.89 0)
+			(effects
+				(font
+					(size 1.27 1.27)
+				)
+				(hide yes)
+			)
+		)
+		(property "Description" ""
+			(at 102.87 135.89 0)
+			(effects
+				(font
+					(size 1.27 1.27)
+				)
+				(hide yes)
+			)
+		)
+		(pin "8"
+		)
+		(pin "5"
+		)
+		(pin "6"
+		)
+		(pin "2"
+		)
+		(pin ""
+		)
+		(pin "1"
+		)
+		(pin "7"
+		)
+		(pin "4"
+		)
+		(instances
+			(project ""
+				(path "/6b7edb0b-ba84-49d7-8a33-d453b93ff911"
+					(reference "LiMa-Kontroller1")
+					(unit 1)
+				)
